File: Hardware/KiCAD Projects/FOC_DRV8323/FOC_DRV8323.kicad_sch (KiCad schematic)
At the start: 12 parts, among them J101 PZ254-1-13-Z-8.5, J102 PZ254-1-13-Z-8.5, J103 MKS Power, Q101 HSBB6066, U101 LIS2DE12

Commit message: Hardware update
- Removed 5V net as it is not really needed for typical SimpleFOC encoders. This reduces part cost a lot.
- Fixed SPI pin assignment
- Exposed another GPIO pin in place of the +5V pin
- Boards changed to transfer power via the standoff pads instead of a solder connection
- Moved accelerometer to the controller board
- Resistance changes to reduce BOM
- Replaced encoder connection with JST-XH
Parts:
- removed C101, C102: 1u, Capacitor_SMD:C_0603_1608Metric, symbol Device:C
- removed J103: MKS Power, TestPoint:TestPoint_2Pads_Pitch5.08mm_Drill1.3mm, symbol Connector:Conn_01x02_Pin
- removed U101: LIS2DE12, Package_LGA:LGA-12_2x2mm_P0.5mm, symbol Sensor_Motion:LIS2DE12
- added H101, H102, H103, H104: MountingHole_Pad, MountingHole:MountingHole_3.2mm_M3_Pad_Via, symbol Mechanical:MountingHole_Pad
- added R106: 1k, Resistor_SMD:R_0603_1608Metric, symbol Device:R
- added TH101: NTCS0805E3103JMT, Resistor_SMD:R_0805_2012Metric, symbol Device:Thermistor_NTC
- J101: footprint Connector_PinHeader_2.54mm:PinHeader_1x14_P2.54mm_Vertical_SMD_Pin1Left -> Connector_PinHeader_2.54mm:PinHeader_1x13_P2.54mm_Vertical_SMD_Pin1Left
- J102: footprint Connector_PinHeader_2.54mm:PinHeader_1x14_P2.54mm_Vertical_SMD_Pin1Left -> Connector_PinHeader_2.54mm:PinHeader_1x13_P2.54mm_Vertical_SMD_Pin1Right
Connections:
- net +3V3: now also R106.2
- net Driver 1/ENABLE: now also J101.6 (Pin_6); no longer J101.7 (Pin_7)
- net Driver 1/nFAULT: now also J101.7 (Pin_7); no longer J101.6 (Pin_6)
- net GND: now also H102.1, H104.1, TH101.2
- net VM: now also H101.1, H103.1
- net at J102.11 (Pin_11): now also R106.1, TH101.1
- net +5V: no longer names the net of J101.12 (Pin_12)
- no-connect marks 3 -> 2

Commit message: Driver redesign to allow 8323H and 8323S
Parts:
- added R107: 1k, Resistor_SMD:R_0603_1608Metric, symbol Device:R
- added R108, R109, R110: 0, Resistor_SMD:R_0603_1608Metric, symbol Device:R
Connections:
- net Driver 1/SOA is gone; now on net HDR2_09_Thermistor: J102.9 (Pin_9)
- net +3V3: now also R107.2
- net HDR2_09_Thermistor: now reaches R106.1, TH101.1
- net HDR2_09_Thermistor: no longer J102.11 (Pin_11)
- net BrakeChop renamed HDR1_10_Drv1Fault
- net HDR1_10_Drv1Fault: no longer R101.1
- net Driver 0/CAL renamed HDR2_02_BrakeChop
- net HDR2_02_BrakeChop: now also R101.1
- net Driver 0/ENABLE renamed HDR1_09_Drv1Select
- net Driver 0/INHA renamed HDR2_08_Drv0INHA
- net Driver 0/INHB renamed HDR2_07_Drv0INHB
- net Driver 0/INHC renamed HDR2_06_Drv0INHC
- net Driver 0/SOA renamed HDR2_12_Drv0SOA
- net Driver 0/SOB renamed HDR2_13_Drv0SOB
- net Driver 0/SPI_SCLK renamed HDR1_03_SCLK
- net HDR1_03_SCLK: now also R108.2
- net Driver 0/SPI_SDI renamed HDR1_05_MOSI
- net HDR1_05_MOSI: now also R110.2
- net Driver 0/SPI_SDO renamed HDR1_04_MISO
- net HDR1_04_MISO: now also R107.1, R109.2
- net Driver 0/SPI_nSCS renamed HDR1_02_Drv0Enable
- net Driver 0/nFAULT renamed HDR1_08_Drv1Enable
- net Driver 1/ENABLE renamed HDR1_06_Drv0Fault
- net Driver 1/INHA renamed HDR2_05_Drv1INHA
- net Driver 1/INHB renamed HDR2_04_Drv1INHB
- net Driver 1/INHC renamed HDR2_03_Drv1INHC
- net Driver 1/SOB renamed HDR2_10_Drv1SOA
- net Driver 1/SPI_nSCS renamed HDR1_01_Drv0Select
- net Driver 1/nFAULT renamed HDR1_07_Calibrate
- new net Driver 0/SCLK/VDS: R108.1
- new net Driver 0/SDI/IDRIVE: R110.1
- new net Driver 0/SDO/MODE: R109.1
- new net HDR2_11_Drv1SOB: J102.11 (Pin_11)
Other:
- sheet Driver 0 ports: added SCLK/VDS, SDI/IDRIVE, SDO/MODE, nSCS/GAIN; removed SPI_SCLK, SPI_SDI, SPI_SDO, SPI_nSCS
- sheet Driver 1 ports: added SCLK/VDS, SDI/IDRIVE, SDO/MODE, nSCS/GAIN; removed SPI_SCLK, SPI_SDI, SPI_SDO, SPI_nSCS
- note added: "Bus connectors for -S version Do not populate for -H version"
- note added: "SPI Pullup for -S version Do not populate for -H version"
- moved on the sheet: H101, H102, H103, H104, J101, J102, R106, TH101
