File: Hardware/KiCAD Projects/FOC_DRV8323/drv1.kicad_sch (KiCad schematic)
At the start: 21 parts, among them J201 DB301V-3.5-3P-GN-S, Q201 HSBB6066, Q202 HSBB6066, Q203 HSBB6066, Q204 HSBB6066, Q205 HSBB6066, Q206 HSBB6066, U201 DRV8323S

Commit message: Driver redesign to allow 8323H and 8323S
Parts:
- added R206, R209: 47k, Resistor_SMD:R_0603_1608Metric, symbol Device:R
- added R207: 0, Resistor_SMD:R_0603_1608Metric, symbol Device:R
- R201: value 1k -> 75k
Connections:
- net DVDD: now also R207.2; no longer R201.1
- net GND: now also R201.2, R206.2, R209.2
- net SPI_SCLK renamed SCLK/VDS
- net SCLK/VDS: now also R201.1
- net SPI_SDI renamed SDI/IDRIVE
- net SDI/IDRIVE: now also R207.1
- net SPI_SDO renamed SDO/MODE
- net SDO/MODE: now also R206.1; no longer R201.2
- net SPI_nSCS renamed nSCS/GAIN
- net nSCS/GAIN: now also R209.1
Other:
- note added: "Configuration for -H version Do not populate for -S version"
- note added: "MODE: 3 PWM IDRIVE: Max VDS: SFault at 0.26V ~50A GAIN: 10V/V -> ADC saturates at 30A"
- moved on the sheet: C201, C202, C203, C204, C205, C206, C207, C208, J201, Q201, Q202, Q203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
