File: Hardware/KiCAD Projects/FOC_RP2350/comms.kicad_sch (KiCad schematic)
At the start: 12 parts, among them SW301 DSHP04TSGER, U301 THVD1424RGTR

Commit message: Hardware update
- Removed 5V net as it is not really needed for typical SimpleFOC encoders. This reduces part cost a lot.
- Fixed SPI pin assignment
- Exposed another GPIO pin in place of the +5V pin
- Boards changed to transfer power via the standoff pads instead of a solder connection
- Moved accelerometer to the controller board
- Resistance changes to reduce BOM
- Replaced encoder connection with JST-XH
Parts:
- removed TH301: NTCS0805E3103JMT, Resistor_SMD:R_0805_2012Metric, symbol Device:Thermistor_PTC
- added C301, C302: 1u, Capacitor_SMD:C_0603_1608Metric, symbol Device:C
- added D303: KT-0805G, LED_SMD:LED_0805_2012Metric, symbol Device:LED
- added U302: LIS2DE12, Package_LGA:LGA-12_2x2mm_P0.5mm, symbol Sensor_Motion:LIS2DE12
- R301: value 4.7k -> 1k
- R302, R303: value 680 -> 1k
- R304, R305, R306, R307: value 4.7k -> 5.1k
Connections:
- net 3V3: now also C301.1, C302.1, D303.2 (A), U302.10 (Vdd_IO), U302.9 (Vdd); no longer R301.1
- net GND: now also R301.1, C301.2, C302.2, U302.5 (RES), U302.6 (GND), U302.7 (GND), U302.8 (GND)
- net Board Temp: no longer names the net of R301.2
- net Board Temp: now also D303.1 (K)
- new net Accel_CS: U302.2 (~{CS})
- new net Accel_SCL: U302.1 (SCL/SPC)
- new net Accel_SDI: U302.4 (SDA/SDI)
- new net Accel_SDO: U302.3 (SA0/SDO)
- no-connect marks 1 -> 3
Other:
- note added: "Accelerometer & Temp Sensor"
- note added: "RS-422/485 Com Bus"
- note added: "Status LEDs"
- note removed: "RS-485 Com Bus"
- moved on the sheet: D301, D302, R302, R303

Commit message: Driver redesign to allow 8323H and 8323S
Parts:
- removed C301, C302: 1u, Capacitor_SMD:C_0603_1608Metric, symbol Device:C
- removed U302: LIS2DE12, Package_LGA:LGA-12_2x2mm_P0.5mm, symbol Sensor_Motion:LIS2DE12
- added D304: KT-0805R, LED_SMD:LED_0805_2012Metric, symbol Device:LED
- added R308: 1k, Resistor_SMD:R_0805_2012Metric, symbol Device:R
Connections:
- net GND: now also R308.1
- new net: D304.1 (K), R308.2
- new net Led3: D304.2 (A)
- no-connect marks 3 -> 1
Other:
- note removed: "Accelerometer & Temp Sensor"
